File: microUnUn/microUnUn.kicad_pcb (KiCad board)
At the start: 2 copper layers, 30.8 x 24.4 mm, 6 parts, among them J1 BNC, U1 Core

Commit message: Add files via upload
Parts:
- added REF**: MountingHole_2.5mm, MountingHole:MountingHole_2.5mm, F.Cu at (110.6, 70.7)
Changed lines of the file:
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@@
   (net 3 "Net-(J2-Pad1)")
+  (footprint "MountingHole:MountingHole_2.5mm" (layer "F.Cu")
+    (at 110.555221 70.7498)
+    (descr "Mounting Hole 2.5mm, no annular")
+    (tags "mounting hole 2.5mm no annular")
+    (attr exclude_from_pos_files exclude_from_bom)
+    (fp_text reference "REF**" (at 0 -3.5) (layer "F.SilkS") hide
+      (effects (font (size 1 1) (thickness 0.15)))
+    )
+    (fp_text value "MountingHole_2.5mm" (at 0 3.5) (layer "F.Fab") hide
+      (effects (font (size 1 1) (thickness 0.15)))
+    )
+    (fp_text user "${REFERENCE}" (at 0 0) (layer "F.Fab") hide
+      (effects (font (size 1 1) (thickness 0.15)))
+    )
+    (fp_circle (center 0 0) (end 2.5 0) (layer "Cmts.User") (width 0.15) (fill none))
+    (fp_circle (center 0 0) (end 2.75 0) (layer "F.CrtYd") (width 0.05) (fill none))
+    (pad "" np_thru_hole circle (at 0 0) (size 3.2 3.2) (drill 3.2) (layers F&B.Cu *.Mask))
+  )
   (footprint "MountingHole:MountingHole_2.5mm" (layer "F.Cu")
     (at 123.3 70.6)
@@
   (gr_line (start 94.2 66.6) (end 94.2 74.6) (layer "Edge.Cuts") (width 0.1))
   (gr_arc (start 120.1 78.4) (mid 108.432881 82.771366) (end 99.038602 74.587355) (layer "Edge.Cuts") (width 0.1))
-  (gr_text "(cc by-sa 4.0)" (at 115.1 73.7) (layer "B.SilkS")
+  (gr_text "(cc by-sa 4.0)" (at 116.9 73.7) (layer "B.SilkS")
     (effects (font (size 1 1) (thickness 0.25)) (justify mirror))
   )
-  (gr_text "microUnUn" (at 115 67.9) (layer "B.SilkS")
+  (gr_text "microUnUn" (at 116.9 68) (layer "B.SilkS")
     (effects (font (size 1.5 1.5) (thickness 0.3)) (justify mirror))
   )
-  (gr_text "DG1JAN\n2023v1.2" (at 115.1 71.1) (layer "B.SilkS")
+  (gr_text "DG1JAN\n2023v1.2" (at 116.9 71.1) (layer "B.SilkS")
     (effects (font (size 1 1) (thickness 0.25)) (justify mirror))
   )
@@
   )
   (gr_text "GND" (at 123.5 75.9 -90) (layer "F.SilkS")
-    (effects (font (size 1.5 1.5) (thickness 0.3)))
-  )
-  (gr_text "microUnUn" (at 115 70.6) (layer "F.SilkS")
     (effects (font (size 1.5 1.5) (thickness 0.3)))
   )
@@
       )
     )
+  )
+  (zone (net 0) (net_name "") (layer "B.Cu") (hatch edge 0.508)
+    (connect_pads yes (clearance 0))
+    (min_thickness 0.254)
+    (keepout (tracks allowed) (vias allowed) (pads allowed ) (copperpour not_allowed) (footprints allowed))
+    (fill (thermal_gap 0.508) (thermal_bridge_width 0.508))
+    (polygon
+      (pts
+        (xy 120.48 73.096)
+        (xy 110.8 73.096)
+        (xy 110.8 69.43)
+        (xy 120.48 69.43)
+      )
+    )
